Commit message: feat: 碰撞检测添加

File: chapt6/chapt6_ws/src/fishbot_description/urdf/fishbot/actuator/caster.urdf.xacro (robot description, xacro)
@@ -12,4 +12,14 @@
         </material>
       </visual>
+      <!-- 碰撞检测 -->
+      <collision>
+        <origin xyz="0 0 0" rpy="0 0 0"/>
+        <geometry>
+          <sphere radius="0.016"/>
+        </geometry>
+        <material name="yellow">
+          <color rgba="1.0 1.0 0.0 0.8"/>
+        </material>
+      </collision>
     </link>
     <joint name="${caster_name}_caster_joint" type="fixed">

File: chapt6/chapt6_ws/src/fishbot_description/urdf/fishbot/actuator/wheel.urdf.xacro (robot description, xacro)
@@ -12,4 +12,14 @@
         </material>
       </visual>
+      <!-- 碰撞检测 -->
+      <collision>
+        <origin xyz="0 0 0" rpy="1.57079 0 0"/>
+        <geometry>
+          <cylinder length="0.04" radius="0.032"/>
+        </geometry>
+        <material name="yellow">
+          <color rgba="1.0 1.0 0.0 0.8"/>
+        </material>
+      </collision>
     </link>
     <joint name="${wheel_name}_wheel_joint" type="continuous">

File: chapt6/chapt6_ws/src/fishbot_description/urdf/fishbot/base.urdf.xacro (robot description, xacro)
@@ -1,4 +1,5 @@
 <?xml version="1.0"?>
 <robot xmlns:xacro="http://www.ros.org/wiki/xacro">
+  <xacro:include filename="$(find fishbot_description)/urdf/fishbot/common_inertia.xacro"/>
   <xacro:macro name="base_xacro" params="length radius">
     <!-- 底盘 -->
@@ -24,4 +25,15 @@
         </material>
       </visual>
+      <!-- 碰撞属性 -->
+      <collision>
+        <origin xyz="0 0 0" rpy="0 0 0"/>
+        <geometry>
+          <cylinder length="${length}" radius="${radius}"/>
+        </geometry>
+        <material name="white">
+          <color rgba="1.0 1.0 1.0 0.5"/>
+        </material>
+      </collision>
+      <xacro:cylinder_inertia m="1.0" r="${radius}" h="${length}"/>
     </link>
   </xacro:macro>

File: chapt6/chapt6_ws/src/fishbot_description/urdf/fishbot/sensor/camera.urdf.xacro (robot description, xacro)
@@ -12,4 +12,14 @@
         </material>
       </visual>
+      <!-- 碰撞检测 -->
+      <collision>
+        <origin xyz="0 0 0.0" rpy="0 0 0"/>
+        <geometry>
+          <box size="0.02 0.10 0.02"/>
+        </geometry>
+        <material name="green">
+          <color rgba="0.0 1.0 0.0 0.8"/>
+        </material>
+      </collision>
     </link>
     <!-- 机器人相机与身体的连接 -->

File: chapt6/chapt6_ws/src/fishbot_description/urdf/fishbot/sensor/imu.urdf.xacro (robot description, xacro)
@@ -12,4 +12,14 @@
         </material>
       </visual>
+      <!-- 碰撞检测 -->
+      <collision>
+        <origin xyz="0 0 0" rpy="0 0 0"/>
+        <geometry>
+          <box size="0.02 0.02 0.02"/>
+        </geometry>
+        <material name="black">
+          <color rgba="0 0 0 0.8"/>
+        </material>
+      </collision>
     </link>
     <!-- 机器人IMU与身体的连接 -->

File: chapt6/chapt6_ws/src/fishbot_description/urdf/fishbot/sensor/laser.urdf.xacro (robot description, xacro)
@@ -13,4 +13,14 @@
         </material>
       </visual>
+      <!-- 碰撞检测 -->
+      <collision>
+        <origin xyz="0 0 0" rpy="0 0 0"/>
+        <geometry>
+          <cylinder length="0.10" radius="0.01"/>
+        </geometry>
+        <material name="green">
+          <color rgba="0.0 1.0 0.0 0.8"/>
+        </material>
+      </collision>
     </link>
     <joint name="laser_cylinder_joint" type="fixed">
@@ -30,4 +40,14 @@
         </material>
       </visual>
+      <!-- 碰撞检测 -->
+      <collision>
+        <origin xyz="0 0 0" rpy="0 0 0"/>
+        <geometry>
+          <cylinder length="0.02" radius="0.02"/>
+        </geometry>
+        <material name="red">
+          <color rgba="1.0 0.0 0.0 0.8"/>
+        </material>
+      </collision>
     </link>
     <joint name="laser_joint" type="fixed">

Commit message: feat: 添加质量和惯性

File: chapt6/chapt6_ws/src/fishbot_description/urdf/fishbot/actuator/caster.urdf.xacro (robot description, xacro)
@@ -1,4 +1,5 @@
 <?xml version="1.0"?>
 <robot xmlns:xacro="http://www.ros.org/wiki/xacro">
+  <xacro:include filename="$(find fishbot_description)/urdf/fishbot/common_inertia.xacro"/>
   <xacro:macro name="caster_xacro" params="caster_name xyz">
     <link name="${caster_name}_caster_link">
@@ -22,4 +23,5 @@
         </material>
       </collision>
+      <xacro:sphere_inertia m="1.0" r="0.016"/>
     </link>
     <joint name="${caster_name}_caster_joint" type="fixed">

File: chapt6/chapt6_ws/src/fishbot_description/urdf/fishbot/actuator/wheel.urdf.xacro (robot description, xacro)
@@ -1,4 +1,5 @@
 <?xml version="1.0"?>
 <robot xmlns:xacro="http://www.ros.org/wiki/xacro">
+  <xacro:include filename="$(find fishbot_description)/urdf/fishbot/common_inertia.xacro"/>
   <xacro:macro name="wheel_xacro" params="wheel_name xyz">
     <link name="${wheel_name}_wheel_link">
@@ -22,4 +23,5 @@
         </material>
       </collision>
+      <xacro:cylinder_inertia m="1.0" h="0.04" r="0.032"/>
     </link>
     <joint name="${wheel_name}_wheel_joint" type="continuous">

File: chapt6/chapt6_ws/src/fishbot_description/urdf/fishbot/fishbot.urdf (robot description, URDF)
Before this commit: robot fishbot, 10 links, 9 joints
Links:
- link back_caster_link: mass None -> 1.0; geometry collision sphere radius=0.016; visual sphere radius=0.016
- link base_link: mass None -> 1.0; geometry collision cylinder length=0.12 radius=0.1; visual cylinder length=0.12 radius=0.1
- link camera_link: mass None -> 1.0; geometry collision box size=0.02 0.10 0.02; visual box size=0.02 0.10 0.02
- link front_caster_link: mass None -> 1.0; geometry collision sphere radius=0.016; visual sphere radius=0.016
- link imu_link: mass None -> 1.0; geometry collision box size=0.02 0.02 0.02; visual box size=0.02 0.02 0.02
- link laser_cylinder_link: mass None -> 1.0; geometry collision cylinder length=0.10 radius=0.01; visual cylinder length=0.10 radius=0.01
- link laser_link: geometry collision cylinder length=0.02 radius=0.02; visual cylinder length=0.02 radius=0.02
- link left_wheel_link: mass None -> 1.0; geometry collision cylinder length=0.04 radius=0.032; visual cylinder length=0.04 radius=0.032
- link right_wheel_link: mass None -> 1.0; geometry collision cylinder length=0.04 radius=0.032; visual cylinder length=0.04 radius=0.032

File: chapt6/chapt6_ws/src/fishbot_description/urdf/fishbot/sensor/camera.urdf.xacro (robot description, xacro)
@@ -1,4 +1,5 @@
 <?xml version="1.0"?>
 <robot xmlns:xacro="http://www.ros.org/wiki/xacro">
+  <xacro:include filename="$(find fishbot_description)/urdf/fishbot/common_inertia.xacro"/>
   <xacro:macro name="camera_xacro" params="xyz">
     <link name="camera_link">
@@ -22,4 +23,5 @@
         </material>
       </collision>
+      <xacro:box_inertia m="1.0" d="0.02" w="0.10" h="0.02"/>
     </link>
     <!-- 机器人相机与身体的连接 -->

File: chapt6/chapt6_ws/src/fishbot_description/urdf/fishbot/sensor/imu.urdf.xacro (robot description, xacro)
@@ -1,4 +1,5 @@
 <?xml version="1.0"?>
 <robot xmlns:xacro="http://www.ros.org/wiki/xacro">
+  <xacro:include filename="$(find fishbot_description)/urdf/fishbot/common_inertia.xacro"/>
   <xacro:macro name="imu_xacro" params="xyz">
     <link name="imu_link">
@@ -22,4 +23,5 @@
         </material>
       </collision>
+      <xacro:box_inertia m="1.0" d="0.02" w="0.02" h="0.02"/>
     </link>
     <!-- 机器人IMU与身体的连接 -->

File: chapt6/chapt6_ws/src/fishbot_description/urdf/fishbot/sensor/laser.urdf.xacro (robot description, xacro)
@@ -1,4 +1,5 @@
 <?xml version="1.0"?>
 <robot xmlns:xacro="http://www.ros.org/wiki/xacro">
+  <xacro:include filename="$(find fishbot_description)/urdf/fishbot/common_inertia.xacro"/>
   <xacro:macro name="laser_xacro" params="xyz">
     <!-- 雷达支撑杆 -->
@@ -23,4 +24,5 @@
         </material>
       </collision>
+      <xacro:cylinder_inertia m="1.0" h="0.10" r="0.01"/>
     </link>
     <joint name="laser_cylinder_joint" type="fixed">

Commit message: feat: gazebo标签扩展修改颜色

File: chapt6/chapt6_ws/src/fishbot_description/urdf/fishbot/actuator/caster.urdf.xacro (robot description, xacro)
@@ -3,4 +3,7 @@
   <xacro:include filename="$(find fishbot_description)/urdf/fishbot/common_inertia.xacro"/>
   <xacro:macro name="caster_xacro" params="caster_name xyz">
+    <gazebo reference="${caster_name}_caster_link">
+      <material>Gazebo/Blue</material>
+    </gazebo>
     <link name="${caster_name}_caster_link">
       <visual>

File: chapt6/chapt6_ws/src/fishbot_description/urdf/fishbot/actuator/wheel.urdf.xacro (robot description, xacro)
@@ -3,4 +3,7 @@
   <xacro:include filename="$(find fishbot_description)/urdf/fishbot/common_inertia.xacro"/>
   <xacro:macro name="wheel_xacro" params="wheel_name xyz">
+    <gazebo reference="${wheel_name}_wheel_link">
+      <material>Gazebo/Blue</material>
+    </gazebo>
     <link name="${wheel_name}_wheel_link">
       <visual>

File: chapt6/chapt6_ws/src/fishbot_description/urdf/fishbot/sensor/camera.urdf.xacro (robot description, xacro)
@@ -3,4 +3,7 @@
   <xacro:include filename="$(find fishbot_description)/urdf/fishbot/common_inertia.xacro"/>
   <xacro:macro name="camera_xacro" params="xyz">
+    <gazebo reference="camera_link">
+      <material>Gazebo/Green</material>
+    </gazebo>
     <link name="camera_link">
       <visual>

File: chapt6/chapt6_ws/src/fishbot_description/urdf/fishbot/sensor/imu.urdf.xacro (robot description, xacro)
@@ -3,4 +3,7 @@
   <xacro:include filename="$(find fishbot_description)/urdf/fishbot/common_inertia.xacro"/>
   <xacro:macro name="imu_xacro" params="xyz">
+    <gazebo reference="imu_link">
+      <material>Gazebo/Black</material>
+    </gazebo>
     <link name="imu_link">
       <visual>

File: chapt6/chapt6_ws/src/fishbot_description/urdf/fishbot/sensor/laser.urdf.xacro (robot description, xacro)
@@ -3,4 +3,10 @@
   <xacro:include filename="$(find fishbot_description)/urdf/fishbot/common_inertia.xacro"/>
   <xacro:macro name="laser_xacro" params="xyz">
+    <gazebo reference="laser_cylinder_link">
+      <material>Gazebo/Black</material>
+    </gazebo>
+    <gazebo reference="laser_link">
+      <material>Gazebo/Black</material>
+    </gazebo>
     <!-- 雷达支撑杆 -->
     <link name="laser_cylinder_link">
