Commit message: feat: 机械臂建模完善

File: practice/src/arm1/urdf/robot_arm.urdf (robot description, URDF)
Before this commit: robot arm, 7 links, 6 joints
Links:
- added link hand_left_link, mass 1; collision box size=0.1 0.2 0.05; visual box size=0.1 0.05 0.1
- added link hand_right_link, mass 1; collision box size=0.1 0.2 0.05; visual box size=0.1 0.05 0.1
Joints:
- added joint hand_left_joint: type prismatic, parent gripper_base_link, child hand_left_link, origin xyz=0.0 -0.075 0.05 rpy=0 0 0, axis 0 1 0, limit lower=0 upper=0.05 effort=100 velocity=1, mimic joint=hand_right_joint
- added joint hand_right_joint: type prismatic, parent gripper_base_link, child hand_right_link, origin xyz=0.0 0.075 0.05 rpy=0 0 0, axis 0 -1 0, limit lower=0 upper=0.05 effort=100 velocity=1
