Commit message: feat: 添加相机支架

File: practice/src/dobot/urdf/cr3_robot_full.urdf (robot description, URDF)
Before this commit: robot cr3_robot, 10 links, 8 joints
Links:
- added link camera_bracket, mass 0.653; collision box size=0.06 0.06 0.2; visual box size=0.06 0.06 0.2
Joints:
- added joint camera_bracket_joint: type fixed, parent pillar_body, child camera_bracket, origin xyz=0 0 0.6 rpy=0 0 0
