Commit message: feat: 代码完善

File: practice/src/dobot/urdf/cr3_robot_full.ros2.urdf (robot description, URDF)
Before this commit: robot cr3_robot, 10 links, 9 joints
Links:
- link Link1: geometry collision mesh filename=package://dobot/mesh/Link1.STL; visual mesh filename=package://dobot/mesh/Link1.STL
- link Link2: geometry collision mesh filename=package://dobot/mesh/Link2.STL; visual mesh filename=package://dobot/mesh/Link2.STL
- link Link3: geometry collision mesh filename=package://dobot/mesh/Link3.STL; visual mesh filename=package://dobot/mesh/Link3.STL
- link Link4: geometry collision mesh filename=package://dobot/mesh/Link4.STL; visual mesh filename=package://dobot/mesh/Link4.STL
- link Link5: geometry collision mesh filename=package://dobot/mesh/Link5.STL; visual mesh filename=package://dobot/mesh/Link5.STL
- link Link6: geometry collision mesh filename=package://dobot/mesh/Link6.STL; visual mesh filename=package://dobot/mesh/Link6.STL
- link base_link: geometry collision mesh filename=package://dobot/mesh/base_link.STL; visual mesh filename=package://dobot/mesh/base_link.STL
