Commit message: feat: 夹爪模型完善

File: practice/src/dobot/urdf/cr3_robot_gripper.urdf (robot description, URDF)
Before this commit: robot cr3_robot, 10 links, 9 joints
Links:
- added link gripper_link, mass 0.1; collision mesh filename=../mesh/Gripper.stl scale=0.001 0.001 0.001; visual mesh filename=../mesh/Gripper.stl scale=0.001 0.001 0.001
- link flange_link: geometry collision mesh filename=../mesh/Flange.stl scale=0.001 0.001 0.001; visual mesh filename=../mesh/Flange.stl scale=0.001 0.001 0.001
Joints:
- added joint joint_gripper: type fixed, parent flange_link, child gripper_link, origin xyz=0 0.05 0 rpy=0 0 0, axis 0 0 0, limit lower=-6.27 upper=6.27 effort=0 velocity=0
